Commit message: cleanup

File: multi_jackal_description/urdf/accessories/bridge_plate.urdf.xacro (robot description, xacro)
@@ -11,5 +11,5 @@
         <origin xyz="0 0 0" rpy="1.5707 0.0 1.5707" />
         <geometry>
-          <mesh filename="package://my_jackal_description/meshes/bridge-plate.stl"/>
+          <mesh filename="package://multi_jackal_description/meshes/bridge-plate.stl"/>
         </geometry>
         <material name="dark_grey" />

File: multi_jackal_description/urdf/accessories/camera_mount.urdf.xacro (robot description, xacro)
@@ -6,5 +6,5 @@
         <origin xyz="0 0 0" rpy="1.5707 0 1.5707" />
         <geometry>
-          <mesh filename="package://my_jackal_description/meshes/camera-bracket.stl" scale="0.001 0.001 0.001" />
+          <mesh filename="package://multi_jackal_description/meshes/camera-bracket.stl" scale="0.001 0.001 0.001" />
         </geometry>
         <material name="dark_grey" />
@@ -15,5 +15,5 @@
         <origin xyz="0 0 0" rpy="0 0 1.5707" />
         <geometry>
-          <mesh filename="package://my_jackal_description/meshes/camera-beam.stl" scale="0.001 0.001 0.001" />
+          <mesh filename="package://multi_jackal_description/meshes/camera-beam.stl" scale="0.001 0.001 0.001" />
         </geometry>
         <material name="dark_grey" />

File: multi_jackal_description/urdf/accessories/novatel_smart6.urdf.xacro (robot description, xacro)
@@ -6,5 +6,5 @@
       <origin xyz="0 0 0" rpy="0 0 0" />
       <geometry>
-        <mesh filename="package://my_jackal_description/meshes/novatel-smart6.stl"/>
+        <mesh filename="package://multi_jackal_description/meshes/novatel-smart6.stl"/>
       </geometry>
       <material name="novatel_white">

File: multi_jackal_description/urdf/accessories/sick_lms1xx_mount.urdf.xacro (robot description, xacro)
@@ -28,5 +28,5 @@
   <xacro:include filename="$(find lms1xx)/urdf/sick_lms1xx.urdf.xacro" />
   <xacro:macro name="sick_lms1xx_mount" params="prefix topic">
-    <sick_lms1xx frame="${prefix}_laser" topic="${topic}" />
+    <sick_lms1xx frame="${prefix}_laser" topic="${topic}" robot_namespace="$(arg namespace)" />
     <link name="${prefix}_laser_mount">
       <visual>
@@ -34,5 +34,5 @@
         <geometry>
           <!-- Origin of this mesh is the base of the bracket. -->
-          <mesh filename="package://my_jackal_description/meshes/sick-lms1xx-bracket.stl" />
+          <mesh filename="package://multi_jackal_description/meshes/sick-lms1xx-bracket.stl" />
         </geometry>
         <material name="dark_grey" />

File: multi_jackal_description/urdf/accessories/twocams.urdf.xacro (robot description, xacro)
@@ -1,4 +1,5 @@
 <?xml version="1.0"?>
 <robot >
+  <!-- Front camera. -->
   <joint name="front_camera_mount_joint" type="fixed">
     <origin xyz="0.060 0 0" rpy="0 0 0" />
@@ -22,4 +23,5 @@
     <child link="front_camera" />
   </joint>
+  <!-- Rear camera. INCOMPLETE, NO IMAGE CREATED.-->
   <joint name="rear_camera_mount_joint" type="fixed">
     <origin xyz="0 0 0" rpy="0 0 0" />

File: multi_jackal_description/urdf/base_accessories.urdf.xacro (robot description, xacro)
@@ -1,12 +1,4 @@
 <?xml version="1.0"?>
 <robot xmlns:xacro="http://www.ros.org/wiki/xacro">
-  <!--
-    As you add to this URDF, please be aware that both the robot and
-    simulation include it. You must retain compatibility with all of
-    the following launch files:
-    jackal_viz/launch/view_model.launch
-    jackal_gazebo/launch/jackal_world.launch
-    jackal_base/launch/base.launch
-  -->
   <!-- Macros to generate standoffs for offset payload mounting. -->
   <xacro:include filename="accessories/standoffs.urdf.xacro" />
@@ -17,5 +9,5 @@
   <xacro:if value="$(optenv JACKAL_LASER 0)">
     <sick_lms1xx_mount prefix="$(optenv JACKAL_LASER_MOUNT front)"
-                       topic="$(optenv JACKAL_LASER_TOPIC front/scan)"/>
+                       topic="$(arg namespace)/$(optenv JACKAL_LASER_TOPIC front/scan)"/>
     <joint name="$(optenv JACKAL_LASER_MOUNT front)_laser_mount_joint" type="fixed">
       <origin xyz="$(optenv JACKAL_LASER_OFFSET 0 0 0)"

File: multi_jackal_description/urdf/jackal.urdf.xacro (robot description, xacro)
@@ -1,20 +1,24 @@
 <?xml version="1.0"?>
+<!-- This URDF should be loaded into a ROS parameter using xacro, then loaded
+     into Gazebo using robot state publisher.
+     Requires the arguments: $namespace, $id -->
 <robot name="jackal" xmlns:xacro="http://www.ros.org/wiki/xacro">
-  <xacro:property name="PI" value="3.1415926535897931" />
-  <xacro:property name="wheelbase" value="0.262" />
-  <xacro:property name="track" value="0.37559" />
-  <xacro:property name="wheel_vertical_offset" value="0.0345" />
+  <xacro:property name="PI"                        value="3.1415926535897931" />
+  <xacro:property name="wheelbase"                 value="0.262" />
+  <xacro:property name="track"                     value="0.37559" />
+  <xacro:property name="wheel_vertical_offset"     value="0.0345" />
   <xacro:property name="footprint_vertical_offset" value="-0.0655" />
-  <xacro:property name="wheel_radius" value="0.098" />
-  <xacro:property name="wheel_width" value="0.040" />
-  <xacro:property name="chassis_length" value="0.420" />
-  <xacro:property name="chassis_width" value="0.310" />
-  <xacro:property name="chassis_height" value="0.184" />
-  <xacro:property name="dummy_inertia" value="1e-09"/>
-  <xacro:property name="mount_spacing" value="0.120" />
-  <material name="dark_grey"><color rgba="0.2 0.2 0.2 1.0" /></material>
+  <xacro:property name="wheel_radius"              value="0.098" />
+  <xacro:property name="wheel_width"               value="0.040" />
+  <xacro:property name="chassis_length"            value="0.420" />
+  <xacro:property name="chassis_width"             value="0.310" />
+  <xacro:property name="chassis_height"            value="0.184" />
+  <xacro:property name="dummy_inertia"             value="1e-09"/>
+  <xacro:property name="mount_spacing"             value="0.120" />
+  <material name="dark_grey"><color rgba=" 0.2 0.2 0.2 1.0" /></material>
   <material name="light_grey"><color rgba="0.4 0.4 0.4 1.0" /></material>
   <material name="yellow"><color rgba="0.8 0.8 0.0 1.0" /></material>
   <material name="black"><color rgba="0.15 0.15 0.15 1.0" /></material>
+  <!-- The wheel template. -->
   <xacro:macro name="wheel" params="prefix *joint_pose">
     <link name="${prefix}_wheel_link">
@@ -62,4 +66,5 @@
     </transmission>
   </xacro:macro>
+  <!-- The joints and links. -->
   <xacro:wheel prefix="front_left">
     <origin xyz="${wheelbase/2} ${track/2} ${wheel_vertical_offset}" rpy="0 0 0" />
@@ -166,20 +171,9 @@
     <origin xyz="${mount_spacing} 0 0" />
   </joint>
-  <!-- Adding AR tag. -->
-  <xacro:if value="$(arg tagged)">
-    <xacro:include filename="$(find tag_world)/models/tag_box2.urdf.xacro"/>
-  </xacro:if>
-  <!-- End adding AR tag. -->
   <!-- Bring in simulation data for Gazebo. -->
   <xacro:include filename="jackal.gazebo" />
-  <!-- Optional standard accessories, including their simulation data. The rendering
-       of these into the final description is controlled by optenv variables, which
-       default each one to off.-->
-  <xacro:include filename="accessories.urdf.xacro" />
-  <!-- Adding additional cameras. -->
-  <xacro:unless value="$(arg tagged)">
-    <xacro:include filename="jackal_extras.urdf.xacro"/>
-  </xacro:unless>
-  <!-- Optional custom includes. -->
-  <xacro:include filename="$(optenv JACKAL_URDF_EXTRAS empty.urdf)" />
+  <!-- Optional standard accessories, as supplied by Clearpath.-->
+  <xacro:include filename="base_accessories.urdf.xacro" />
+  <!-- Optional custom accessories. -->
+  <xacro:include filename="custom_accessories.urdf.xacro" />
 </robot>
